File: pcb/dna/dna.kicad_pcb (KiCad board)
At the start: 2 copper layers, 227 x 100 mm, 62 parts, among them J1 AudioPlug3, SW1 RotaryEncoder, SW2 RotaryEncoder, SW3 RotaryEncoder, SW4 RotaryEncoder, SW5 RotaryEncoder, SW6 RotaryEncoder, SW7 RotaryEncoder, SW8 RotaryEncoder, U1 MCP23018x-x-SO

Commit message: Update PCB source files
Parts:
- D1, D10, D11, D12, D13, D14, D15, D16, D17, D18, D19, D2, D20, D21, D22, D3, D4, D5, D6, D7, D8, D9: footprint Diode_SMD:D_SOD-123 -> Diode_THT:D_DO-35_SOD27_P7.62mm_Horizontal
- R1, R2: footprint Resistor_SMD:R_0805_2012Metric -> Resistor_THT:R_Axial_DIN0207_L6.3mm_D2.5mm_P7.62mm_Horizontal
- SW1, SW2, SW3, SW4, SW5, SW6, SW7, SW8: footprint Rotary_Encoder:RotaryEncoder_Bourns_Vertical_PEC12R-3x17F-Sxxxx -> Rotary_Encoder:RotaryEncoder_Bourns_Vertical_PEC12R-3x17F-Nxxxx
- U1: value MCP23018x-x-SO -> MCP23018x-x-SP; footprint Package_SO:SOIC-28W_7.5x17.9mm_P1.27mm -> Package_DIP:DIP-28_W7.62mm
- moved U1 25.4 mm to (203.7, 41.9)
- moved D11 9.01 mm to (261.1, 84.9), turned to 90 degrees
- moved D8 8.98 mm to (196.8, 84.9), turned to 90 degrees
- moved D19 8.98 mm to (196.8, 104.0), turned to 90 degrees
- moved D22 8.95 mm to (261.1, 104.0), turned to 90 degrees
- moved D9 6.91 mm to (223.0, 84.9), turned to 90 degrees
- moved D20 6.91 mm to (223.0, 104.0), turned to 90 degrees
- moved D21 6.91 mm to (242.1, 104.0), turned to 90 degrees
- moved D1 6.91 mm to (55.6, 84.9), turned to 90 degrees
- moved D2 6.91 mm to (74.6, 84.9), turned to 90 degrees
- moved D3 6.91 mm to (93.7, 84.9), turned to 90 degrees
- moved D6 6.91 mm to (150.8, 84.9), turned to 90 degrees
- moved D7 6.91 mm to (169.9, 84.9), turned to 90 degrees
- moved D12 6.91 mm to (55.6, 104.0), turned to 90 degrees
- moved D13 6.91 mm to (74.6, 104.0), turned to 90 degrees
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Routing:
- net +3V3: track 258.5 -> 235.0 mm, vias 2 -> 0
- net ENC0_A: track 94.8 -> 109.6 mm
- net ENC4_A: track 113.0 -> 127.5 mm
- net ENC0_B: track 97.5 -> 111.0 mm
- net ENC4_B: track 105.6 -> 118.4 mm
- net ENC1_A: track 72.6 -> 84.9 mm
- net ENC5_A: track 91.7 -> 102.8 mm
- net ENC1_B: track 75.3 -> 86.3 mm
- net ENC2_A: track 50.4 -> 60.2 mm
- net ENC5_B: track 84.2 -> 93.7 mm
- net ENC2_B: track 53.1 -> 61.5 mm
- net ENC6_A: track 69.8 -> 77.6 mm
- net ENC3_A: track 28.2 -> 35.4 mm
- net MIDI_SINK: track 29.0 -> 22.3 mm
- net ENC6_B: track 62.4 -> 68.5 mm
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