File: pcb/dna/dna.kicad_sch (KiCad schematic)
At the start: 58 parts, among them J1 AudioPlug3, SW1 RotaryEncoder, SW2 RotaryEncoder, SW3 RotaryEncoder, SW4 RotaryEncoder, SW5 RotaryEncoder, SW6 RotaryEncoder, SW7 RotaryEncoder, SW8 RotaryEncoder, U1 MCP23018x-x-SO

Commit message: Update PCB source files
Parts:
- removed U1: MCP23018x-x-SO, Package_SO:SOIC-28W_7.5x17.9mm_P1.27mm, symbol Interface_Expansion:MCP23018x-x-SO
- added U1: MCP23018x-x-SP, Package_DIP:DIP-28_W7.62mm, symbol Interface_Expansion:MCP23018x-x-SP
- D1, D10, D11, D12, D13, D14, D15, D16, D17, D18, D19, D2, D20, D21, D22, D3, D4, D5, D6, D7, D8, D9: footprint Diode_SMD:D_SOD-123 -> Diode_THT:D_DO-35_SOD27_P7.62mm_Horizontal
- R1, R2: footprint Resistor_SMD:R_0805_2012Metric -> Resistor_THT:R_Axial_DIN0207_L6.3mm_D2.5mm_P7.62mm_Horizontal
- SW1, SW2, SW3, SW4, SW5, SW6, SW7, SW8: footprint Rotary_Encoder:RotaryEncoder_Bourns_Vertical_PEC12R-3x17F-Sxxxx -> Rotary_Encoder:RotaryEncoder_Bourns_Vertical_PEC12R-3x17F-Nxxxx
Connections:
- net +3V3: now also U1.11 (V_{DD}), U1.16 (~{RESET})
- net ENC0_A: now also U1.3 (GPB0)
- net ENC0_B: now also U1.4 (GPB1)
- net ENC1_A: now also U1.5 (GPB2)
- net ENC1_B: now also U1.6 (GPB3)
- net ENC2_A: now also U1.7 (GPB4)
- net ENC2_B: now also U1.8 (GPB5)
- net ENC3_A: now also U1.9 (GPB6)
- net ENC3_B: now also U1.10 (GPB7)
- net ENC4_A: now also U1.27 (GPA7)
- net ENC4_B: now also U1.26 (GPA6)
- net ENC5_A: now also U1.25 (GPA5)
- net ENC5_B: now also U1.24 (GPA4)
- net ENC6_A: now also U1.23 (GPA3)
- net ENC6_B: now also U1.22 (GPA2)
- net ENC7_A: now also U1.21 (GPA1)
- net ENC7_B: now also U1.20 (GPA0)
- net GND: now also U1.1 (V_{SS}), U1.15 (ADDR)
- net IO_SCL: now also U1.12 (SCL)
- net IO_SDA: now also U1.13 (SDA)
- net PICO_INT: now also U1.19 (INTA)
