File: pcb/dna.kicad_pcb (KiCad board)
At the start: 2 copper layers, 227 x 100 mm, 62 parts, among them J1 AudioPlug3, SW1 RotaryEncoder, SW2 RotaryEncoder, SW3 RotaryEncoder, SW4 RotaryEncoder, SW5 RotaryEncoder, SW6 RotaryEncoder, SW7 RotaryEncoder, SW8 RotaryEncoder, U1 MCP23018x-x-SP

Commit message: Add files via upload
Parts:
- J1: footprint Connector_Audio:Jack_3.5mm_CUI_SJ1-3513N_Horizontal -> Connector_Audio:Jack_3.5mm_CUI_SJ1-3533NG_Horizontal_CircularHoles
- REF** (x4): value MountingHole_2.5mm_Pad -> MountingHole_3mm_Pad; footprint MountingHole:MountingHole_2.5mm_Pad -> MountingHole:MountingHole_3mm_Pad
- SW1, SW2, SW3, SW4, SW5, SW6, SW7, SW8: footprint Rotary_Encoder:RotaryEncoder_Bourns_Vertical_PEC12R-3x17F-Nxxxx -> Rotary_Encoder:RotaryEncoder_Bourns_Vertical_PEC12R-3x17F-Sxxxx
- U1: value MCP23018x-x-SP -> MCP23017x-x-SP
- turned J1 to 90 degrees
Routing:
- net Net-(J1-PadT): track 17.0 -> 20.8 mm
- net Net-(J1-PadR): track 11.3 -> 14.4 mm
